File: pcb/Kretsträd.kicad_pcb (KiCad board)
At the start: 2 copper layers, 112.8 x 95.4 mm, 52 parts, among them J1 Conn_01x02_Female, J2 Conn_01x02_Female, J3 Conn_01x02_Female, J4 Conn_01x02_Female, SW1 SW_PUSH, SW10 SW_PUSH, SW11 SW_PUSH, SW12 SW_PUSH, SW13 SW_PUSH, SW14 SW_PUSH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

Commit message: First PCB production.
Parts:
- moved PWR_SW_1 5.45 mm to (183.6, 130.2)
- moved PWR_SW_2 5.45 mm to (183.6, 130.2)
- moved TH_PCB_3 4.08 mm to (187.2, 122.6)
- moved D17 2.05 mm to (162.6, 111.5), turned to -90 degrees
- moved D16 1.79 mm to (159.9, 111.5), turned to -90 degrees
- moved TH1 1.40 mm to (96.7, 55.7)
- moved SW11 1.22 mm to (89.4, 100.6)
- moved D1 1.22 mm to (97.7, 67.9)
- moved D11 1.22 mm to (97.7, 101.9)
- moved D6 1.22 mm to (97.7, 84.9)
- moved SW1 1.22 mm to (89.4, 66.6)
- moved SW6 1.22 mm to (89.4, 83.6)
- moved J1 1.08 mm to (167.7, 114.6), turned to 110 degrees
- moved J2 1.08 mm to (167.7, 114.6), turned to -70 degrees
- moved TH5 1.06 mm to (164.3, 124.4)
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- renumbered TH5 to TH4, TH4 to TH5
Connections:
- SW10 pad : col4 -> (no net)
- SW14 pad : col3 -> (no net)
- SW15 pad : col4 -> (no net)
- SW16 pad : col3 -> (no net)
- SW17 pad : col4 -> (no net)
- SW4 pad : col3 -> (no net)
- SW5 pad : col4 -> (no net)
- SW9 pad : col3 -> (no net)
Routing:
- net col3: track 137.6 -> 154.2 mm
- net BT+: track 57.8 -> 64.2 mm
- net /PWR: track 42.0 -> 47.8 mm
- net Net-(D17-Pad2): track 33.8 -> 39.3 mm
- net col4: track 125.0 -> 130.0 mm, vias 6 -> 5
- net Net-(D16-Pad2): track 26.9 -> 30.4 mm, vias 2 -> 1
- net col1: track 137.9 -> 139.4 mm
- net row0: track 103.5 -> 102.3 mm
- net Net-(D8-Pad2): track 26.8 -> 26.3 mm
- net Net-(D3-Pad2): track 27.0 -> 26.5 mm
- net Net-(D13-Pad2): track 27.1 -> 26.5 mm
- net Net-(D9-Pad2): track 26.5 -> 26.0 mm
- net Net-(D14-Pad2): track 26.4 -> 25.9 mm
Other:
- board size 112.8 x 95.4 mm -> 112.2 x 95.8 mm

Commit message: First public version.
Parts:
- removed J4: Conn_01x02_Female, Connector_PinSocket_2.54mm:PinSocket_1x02_P2.54mm_Vertical
- moved TH_PCB_1 2.80 mm to (176.0, 93.0)
- moved TH_PCB_2 2.68 mm to (188.6, 93.0)
- moved G*** 2.02 mm to (109.3, 111.9)
- moved TH2 1.87 mm to (155.4, 52.8)
- moved TH3 1.84 mm to (101.2, 107.5)
- moved JP1 1.83 mm to (182.4, 89.4)
- moved D14 1.79 mm to (152.8, 98.4)
- moved D4 1.79 mm to (152.8, 64.4)
- moved D9 1.79 mm to (152.8, 81.4)
- moved SW14 1.79 mm to (144.6, 95.2)
- moved SW16 1.79 mm to (154.6, 120.4)
- moved SW9 1.79 mm to (144.6, 78.2)
- moved D3 1.79 mm to (134.7, 62.2)
- moved SW4 1.79 mm to (144.6, 61.2)
- moved SW5 1.79 mm to (162.6, 63.7)
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Connections:
- SW10 pad : (no net) -> col4
- SW14 pad : (no net) -> col3
- SW15 pad : (no net) -> col4
- SW16 pad : (no net) -> col3
- SW17 pad : (no net) -> col4
- SW4 pad : (no net) -> col3
- SW5 pad : (no net) -> col4
- SW9 pad : (no net) -> col3
Routing:
- net Net-(D17-Pad2): track 39.3 -> 35.4 mm
- net col3: track 154.2 -> 151.3 mm
- net /PWR: track 47.8 -> 49.3 mm
- net row3: track 43.9 -> 45.1 mm, vias 2 -> 4
- net col0: track 155.0 -> 154.4 mm
- net col2: track 118.2 -> 117.6 mm
- net col1: track 139.4 -> 138.8 mm
- net col4: vias 5 -> 7
Other:
- board size 112.2 x 95.8 mm -> 111.6 x 95.3 mm
