File: pcb/Kretsträd.kicad_sch (KiCad schematic)
At the start: 51 parts, among them J1 Conn_01x02_Female, J2 Conn_01x02_Female, J3 Conn_01x02_Female, J4 Conn_01x02_Female, SW1 SW_PUSH, SW10 SW_PUSH, SW11 SW_PUSH, SW12 SW_PUSH, SW13 SW_PUSH, SW14 SW_PUSH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

Commit message: First public version.
Parts:
- removed J4: Conn_01x02_Female, Connector_PinSocket_2.54mm:PinSocket_1x02_P2.54mm_Vertical, symbol Connector:Conn_01x02_Female
- removed TH5: HOLE, MountingHole:MountingHole_3.2mm_M3, symbol SofleKeyboard-rescue:HOLE-Lily58-cache-Lily58_Pro-rescue
Other:
- moved on the sheet: J3
Changed lines of the file:
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@@
   (junction (at 33.528 119.38) (diameter 0) (color 0 0 0 0)
   )
+  (junction (at 50.038 121.92) (diameter 0) (color 0 0 0 0)
+  )
   (junction (at 151.13 38.1) (diameter 0) (color 0 0 0 0)
   )
@@
   (junction (at 212.09 38.1) (diameter 0) (color 0 0 0 0)
   )
-  (junction (at 62.23 121.92) (diameter 0) (color 0 0 0 0)
-  )
-  (junction (at 59.69 121.92) (diameter 0) (color 0 0 0 0)
-  )
   (junction (at 247.65 62.23) (diameter 0) (color 0 0 0 0)
   )
@@
   )
   (junction (at 172.085 38.1) (diameter 0) (color 0 0 0 0)
-  )
-  (junction (at 50.038 121.92) (diameter 0) (color 0 0 0 0)
   )
   (junction (at 187.325 78.74) (diameter 0) (color 0 0 0 0)
@@
     (stroke (width 0) (type default) (color 0 0 0 0))
   )
-  (wire (pts (xy 59.69 124.714) (xy 59.69 121.92))
-    (stroke (width 0) (type default) (color 0 0 0 0))
-  )
-  (wire (pts (xy 62.23 124.714) (xy 62.23 121.92))
-    (stroke (width 0) (type default) (color 0 0 0 0))
-  )
   (wire (pts (xy 172.085 54.61) (xy 171.45 54.61))
     (stroke (width 0) (type default) (color 0 0 0 0))
   )
-  (wire (pts (xy 62.23 121.92) (xy 64.008 121.92))
+  (wire (pts (xy 59.69 124.46) (xy 59.69 126.238))
     (stroke (width 0) (type default) (color 0 0 0 0))
   )
@@
     (stroke (width 0) (type default) (color 0 0 0 0))
   )
+  (wire (pts (xy 50.038 121.92) (xy 59.69 121.92))
+    (stroke (width 0) (type default) (color 0 0 0 0))
+  )
   (polyline (pts (xy 133.096 17.78) (xy 133.096 101.092))
     (stroke (width 0) (type default) (color 0 0 0 0))
@@
   )
   (wire (pts (xy 172.085 38.1) (xy 171.45 38.1))
-    (stroke (width 0) (type default) (color 0 0 0 0))
-  )
-  (wire (pts (xy 50.038 121.92) (xy 59.69 121.92))
     (stroke (width 0) (type default) (color 0 0 0 0))
   )
@@
     )
   )
-  (global_label "GND" (shape input) (at 64.008 121.92 0) (fields_autoplaced)
-    (effects (font (size 1.27 1.27)) (justify left))
-    (property "Intersheet References" "${INTERSHEET_REFS}" (id 0) (at 70.2027 121.9994 0)
-      (effects (font (size 1.27 1.27)) (justify left) hide)
+  (global_label "GND" (shape input) (at 59.69 126.238 270) (fields_autoplaced)
+    (effects (font (size 1.27 1.27)) (justify right))
+    (property "Intersheet References" "${INTERSHEET_REFS}" (id 0) (at 59.6106 132.4327 90)
+      (effects (font (size 1.27 1.27)) (justify right) hide)
     )
   )
@@
     )
     (pin "1")
-  )
-  (symbol (lib_id "SofleKeyboard-rescue:HOLE-Lily58-cache-Lily58_Pro-rescue") (at 97.282 187.452 0) (unit 1)
-    (in_bom yes) (on_board yes)
-    (property "Reference" "TH5" (id 0) (at 97.282 187.452 0)
-      (effects (font (size 1.524 1.524)))
-    )
-    (property "Value" "HOLE" (id 1) (at 97.282 189.992 0)
-      (effects (font (size 1.524 1.524)))
-    )
-    (property "Footprint" "MountingHole:MountingHole_3.2mm_M3" (id 2) (at 97.282 187.452 0)
-      (effects (font (size 1.524 1.524)) hide)
-    )
-    (property "Datasheet" "" (id 3) (at 97.282 187.452 0)
-      (effects (font (size 1.524 1.524)))
-    )
   )
   (symbol (lib_id "Connector:Conn_01x02_Female") (at 106.426 93.345 0) (unit 1)
@@
     )
     (property "Datasheet" "" (id 3) (at 179.07 38.1 0))
-    (pin "1")
-    (pin "2")
-  )
-  (symbol (lib_id "Connector:Conn_01x02_Female") (at 59.69 129.794 90) (mirror x) (unit 1)
-    (in_bom yes) (on_board yes)
-    (property "Reference" "J4" (id 0) (at 61.976 130.81 90)
-      (effects (font (size 1.27 1.27)) (justify left))
-    )
-    (property "Value" "Conn_01x02_Female" (id 1) (at 77.978 132.334 90)
-      (effects (font (size 1.27 1.27)) (justify left))
-    )
-    (property "Footprint" "Connector_PinSocket_2.54mm:PinSocket_1x02_P2.54mm_Vertical" (id 2) (at 59.69 129.794 0)
-      (effects (font (size 1.27 1.27)) hide)
-    )
-    (property "Datasheet" "~" (id 3) (at 59.69 129.794 0)
-      (effects (font (size 1.27 1.27)) hide)
-    )
     (pin "1")
     (pin "2")
@@
     (pin "2")
   )
-  (symbol (lib_id "Connector:Conn_01x02_Female") (at 59.69 116.84 90) (unit 1)
-    (in_bom yes) (on_board yes)
-    (property "Reference" "J3" (id 0) (at 61.976 115.824 90)
+  (symbol (lib_id "Connector:Conn_01x02_Female") (at 64.77 121.92 0) (unit 1)
+    (in_bom yes) (on_board yes)
+    (property "Reference" "J3" (id 0) (at 65.786 124.206 90)
       (effects (font (size 1.27 1.27)) (justify left))
     )
-    (property "Value" "Conn_01x02_Female" (id 1) (at 77.978 114.046 90)
+    (property "Value" "Conn_01x02_Female" (id 1) (at 67.564 140.208 90)
       (effects (font (size 1.27 1.27)) (justify left))
     )
-    (property "Footprint" "Connector_Molex:Molex_PicoBlade_53047-0210_1x02_P1.25mm_Vertical" (id 2) (at 59.69 116.84 0)
-      (effects (font (size 1.27 1.27)) hide)
-    )
-    (property "Datasheet" "~" (id 3) (at 59.69 116.84 0)
+    (property "Footprint" "Connector_Molex:Molex_PicoBlade_53047-0210_1x02_P1.25mm_Vertical" (id 2) (at 64.77 121.92 0)
+      (effects (font (size 1.27 1.27)) hide)
+    )
+    (property "Datasheet" "~" (id 3) (at 64.77 121.92 0)
       (effects (font (size 1.27 1.27)) hide)
     )
@@
       (reference "J3") (unit 1) (value "Conn_01x02_Female") (footprint "Connector_Molex:Molex_PicoBlade_53047-0210_1x02_P1.25mm_Vertical")
     )
-    (path "/a6ed6253-64a5-4e66-a792-ec78a51c9b48"
-      (reference "J4") (unit 1) (value "Conn_01x02_Female") (footprint "Connector_PinSocket_2.54mm:PinSocket_1x02_P2.54mm_Vertical")
-    )
     (path "/6e4bbe2c-1e2d-4539-b6d8-5d5edc57b4de"
       (reference "JP1") (unit 1) (value "to_RAW") (footprint "jw_custom_footprint:SolderJumper-2_P1.3mm_Open_RoundedPad1.0x1.5mm_dual_side")
@@
       (reference "TH4") (unit 1) (value "HOLE") (footprint "MountingHole:MountingHole_3.2mm_M3")
     )
-    (path "/34a97abb-9105-4ea1-827e-4fa7bedd987f"
-      (reference "TH5") (unit 1) (value "HOLE") (footprint "MountingHole:MountingHole_3.2mm_M3")
-    )
     (path "/6f25ff55-ba4b-4316-b506-f9414fe069e3"
