File: rev2/pcb/Kretsträd_v2.kicad_pcb (KiCad board)
At the start: 2 copper layers, 112.5 x 93.1 mm, 49 parts, among them J1 Conn_01x02_Female, J2 Conn_01x02_Female, SW1 SW_PUSH, SW10 SW_PUSH, SW11 SW_PUSH, SW12 SW_PUSH, SW13 SW_PUSH, SW14 SW_PUSH, SW15 SW_PUSH, SW16 SW_PUSH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

Commit message: Rev2 completely redesigned
Parts:
- removed TH_PCB_1, TH_PCB_2, TH_PCB_3: HOLE, MountingHole:MountingHole_2.2mm_M2_Pad
- added Batt_Hole_1: HOLE, MountingHole:MountingHole_2.2mm_M2_ISO14580_Pad, F.Cu at (111.4, 122.8)
- added Batt_Hole_2: HOLE, MountingHole:MountingHole_2.2mm_M2_ISO14580_Pad, F.Cu at (133.6, 119.9)
- added J3: Conn_01x02_Female, Connector_Molex:Molex_Panelmate_53780-0270_1x02-1MP_P1.25mm_Horizontal, F.Cu at (147.9, 107.3)
- added J4: Conn_01x02_Female, Connector_Molex:Molex_Panelmate_53780-0270_1x02-1MP_P1.25mm_Horizontal, B.Cu at (147.9, 107.3)
- SW1: value SW_PUSH -> SW1
- SW10: value SW_PUSH -> SW10
- SW11: value SW_PUSH -> SW11
- SW12: value SW_PUSH -> SW12
- SW13: value SW_PUSH -> SW13
- SW14: value SW_PUSH -> SW14
- SW15: value SW_PUSH -> SW15
- SW16: value SW_PUSH -> SW16
- SW17: value SW_PUSH -> SW17
- SW2: value SW_PUSH -> SW2
- SW3: value SW_PUSH -> SW3
- SW4: value SW_PUSH -> SW4
- SW5: value SW_PUSH -> SW5
- SW6: value SW_PUSH -> SW6
- SW7: value SW_PUSH -> SW7
- SW8: value SW_PUSH -> SW8
- SW9: value SW_PUSH -> SW9
- U1: footprint jw_custom_footprint:Xiao THT jumper pad_flipped -> jw_custom_footprints:Xiao THT jumper pad_big_hole_flipped
- moved U1 93.1 mm to (95.3, 119.1), turned to 97.5 degrees
- moved G*** 65.5 mm to (115.8, 118.4)
- moved J1 35.0 mm to (173.0, 112.6), turned to 165 degrees
- moved J2 35.0 mm to (173.0, 112.6), turned to -15 degrees
- moved Breakaway2 24.6 mm to (136.6, 119.1), turned to -97.5 degrees
- moved D17 16.1 mm to (156.8, 119.3)
- moved Breakaway1 16.0 mm to (108.4, 122.4), turned to -82.5 degrees
- moved D16 15.2 mm to (153.3, 116.4)
- moved D5 14.2 mm to (157.1, 60.4), turned to -90 degrees
- moved PWR_SW_1 11.0 mm to (177.9, 116.8), turned to 75 degrees
- moved PWR_SW_2 11.0 mm to (177.9, 116.8), turned to -105 degrees
- moved D1 8.55 mm to (94.9, 59.9), turned to -90 degrees
- moved SW16 1.78 mm to (147.8, 120.1), turned to 172.5 degrees
- moved TH4 1.76 mm to (159.1, 114.1)
- moved D6 1.76 mm to (94.9, 85.6)
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Connections:
- J1 pad 1: BT+ -> GND
- J1 pad 2: GND -> BT+
- J2 pad 1: BT+ -> GND
- J2 pad 2: GND -> BT+
- SW1 pad 1: col0 -> Net-(D1-A)
- SW1 pad 2: Net-(D1-A) -> col0
- SW5 pad 1: col4 -> Net-(D5-A)
- SW5 pad 2: Net-(D5-A) -> col4
- U1 pad 1: row0 -> row2
- U1 pad 2: col0 -> row0
- U1 pad 3: col1 -> row1
- U1 pad 4: row1 -> col0
- U1 pad 5: col2 -> col4
- U1 pad 7: col4 -> col1
- U1 pad 9: row2 -> col2
Routing:
- net col0: track 163.3 -> 84.5 mm, vias 4 -> 6
- net row3: track 34.9 -> 94.7 mm, vias 1 -> 4
- net RAW: track 69.1 -> 124.6 mm, vias 2 -> 3
- net col1: track 140.0 -> 85.5 mm, vias 5 -> 4
- net row0: track 101.0 -> 152.8 mm, vias 1 -> 3
- net row1: track 99.6 -> 132.6 mm, vias 1 -> 3
- net col4: track 130.1 -> 159.2 mm, vias 5 -> 9
- net col2: track 122.6 -> 101.1 mm, vias 4 -> 7
- net Net-(D16-A): track 37.7 -> 18.1 mm, vias 1 -> 2
- net col3: track 148.3 -> 167.2 mm, vias 5 -> 10
- net BT+: track 53.0 -> 39.3 mm, vias 4 -> 3
- net Net-(D5-A): track 13.6 -> 23.9 mm, vias 1 -> 2
- net unconnected-(U1-PA5_A9_D9_MISO-Pad10)_0: track 9.86 -> 0.00 mm, vias 1 -> 0
- net unconnected-(U1-PA5_A9_D9_MISO-Pad10): track 0.00 -> 9.31 mm, vias 0 -> 1
- net row2: track 106.6 -> 105.0 mm, vias 2 -> 1
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Other:
- board size 112.5 x 93.1 mm -> 103.4 x 89.4 mm
- board text added: "Kretsträd v2 Designed by jw"
- board text removed: "Kretsträd PCB designed by jw"
