File: rev2/pcb/Kretsträd_v2.kicad_sch (KiCad schematic)
At the start: 48 parts, among them J1 Conn_01x02_Female, J2 Conn_01x02_Female, SW1 SW_PUSH, SW10 SW_PUSH, SW11 SW_PUSH, SW12 SW_PUSH, SW13 SW_PUSH, SW14 SW_PUSH, SW15 SW_PUSH, SW16 SW_PUSH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

Commit message: Rev2 completely redesigned
Parts:
- removed TH_PCB_2, TH_PCB_3: HOLE, MountingHole:MountingHole_2.2mm_M2_Pad, symbol SofleKeyboard-rescue:HOLE-Lily58-cache-Lily58_Pro-rescue
- added Batt_Hole_2: HOLE, MountingHole:MountingHole_2.2mm_M2_ISO14580_Pad, symbol SofleKeyboard-rescue:HOLE-Lily58-cache-Lily58_Pro-rescue
- added J3, J4: Conn_01x02_Female, Connector_Molex:Molex_Panelmate_53780-0270_1x02-1MP_P1.25mm_Horizontal, symbol Connector:Conn_01x02_Female
- Batt_Hole_1: renamed from TH_PCB_1; footprint MountingHole:MountingHole_2.2mm_M2_Pad -> MountingHole:MountingHole_2.2mm_M2_ISO14580_Pad
- SW1, SW10, SW11, SW12, SW13, SW14, SW15, SW16, SW17, SW2, SW3, SW4, SW5, SW6, SW7, SW8, SW9: value SW_PUSH -> ${REFERENCE}
- U1: footprint jw_custom_footprint:Xiao THT jumper pad_flipped -> jw_custom_footprints:Xiao THT jumper pad_big_hole_flipped
Connections:
- net BT+: now also J1.2 (Pin_2), J2.2 (Pin_2), J3.2 (Pin_2), J4.2 (Pin_2); no longer J1.1 (Pin_1), J2.1 (Pin_1)
- net GND: now also J1.1 (Pin_1), J2.1 (Pin_1), J3.1 (Pin_1), J4.1 (Pin_1); no longer J1.2 (Pin_2), J2.2 (Pin_2)
- net col0: now also SW1.2, U1.4 (PA11_A3_D3); no longer SW1.1, U1.2 (PA4_A1_D1)
- net col1: now also U1.7 (PB08_A6_D6_TX); no longer U1.3 (PA10_A2_D2)
- net col2: now also U1.9 (PA7_A8_D8_SCK); no longer U1.5 (PA8_A4_D4_SDA)
- net col4: now also SW5.2, U1.5 (PA8_A4_D4_SDA); no longer SW5.1, U1.7 (PB08_A6_D6_TX)
- net row0: now also U1.2 (PA4_A1_D1); no longer U1.1 (PA02_A0_D0)
- net row1: now also U1.3 (PA10_A2_D2); no longer U1.4 (PA11_A3_D3)
- net row2: now also U1.1 (PA02_A0_D0); no longer U1.9 (PA7_A8_D8_SCK)
- net at D5.2 (A): now also SW5.1; no longer SW5.2
- net at D1.2 (A): now also SW1.1; no longer SW1.2
Other:
- moved on the sheet: Batt_Hole_1, Breakaway1, Breakaway2, J1, J2, TH1, TH2, TH3, TH4
