File: rev2/choc/case/Kretsträd_v2.kicad_pcb (KiCad board)
At the start: 2 copper layers, 224.6 x 368.5 mm, 206 parts, among them SW1 SW1, SW10 SW10, SW11 SW11, SW12 SW12, SW13 SW13, SW14 SW14, SW15 SW15, SW16 SW16, SW17 SW17, SW2 SW2, SW3 SW3, SW4 SW4, SW5 SW5, SW6 SW6, SW7 SW7, SW8 SW8, SW9 SW9, U1 SeeeduinoXIAO_nRF52840

Commit message: v2.2
Parts:
- removed the Batt_Hole_1 at (75.0, 307.3)
- removed the Batt_Hole_1 at (231.1, 307.3)
- removed the Batt_Hole_1 at (75.0, 197.3)
- removed the Batt_Hole_1 at (231.1, 197.3)
- removed the Batt_Hole_2 at (97.2, 194.3)
- removed the Batt_Hole_2 at (208.9, 304.3)
- removed the Batt_Hole_2 at (208.9, 194.3)
- removed the Batt_Hole_2 at (97.2, 304.3)
- removed the D1 at (61.4, 246.3)
- removed the D1 at (61.4, 136.3)
- removed the D1 at (244.7, 136.3)
- removed the D1 at (244.7, 246.3)
- removed the D10 at (134.7, 162.5)
- removed the D10 at (134.7, 272.5)
- removed the D10 at (171.3, 272.5)
- removed the D10 at (171.3, 162.5)
- removed the D11 at (61.4, 284.7)
- removed the D11 at (61.4, 174.7)
- removed the D11 at (244.7, 174.7)
- removed the D11 at (244.7, 284.7)
- removed the D12 at (79.9, 281.4)
- removed the D12 at (79.9, 171.4)
- removed the D12 at (226.2, 171.4)
- removed the D12 at (226.2, 281.4)
- removed the D13 at (97.8, 168.7)
- removed the D13 at (97.8, 278.7)
- removed the D13 at (208.3, 278.7)
- removed the D13 at (208.3, 168.7)
- removed the D14 at (116.2, 173.7)
- removed the D14 at (116.2, 283.7)
- removed the D14 at (189.9, 283.7)
- removed the D14 at (189.9, 173.7)
- removed the D15 at (134.6, 289.0)
- removed the D15 at (134.6, 179.0)
- removed the D15 at (171.4, 179.0)
- removed the D15 at (171.4, 289.0)
- removed the D16 at (119.6, 307.7)
- removed the D16 at (119.6, 197.7)
- removed the D16 at (186.4, 307.7)
- removed the D16 at (186.4, 197.7)
- removed the D17 at (122.6, 198.2)
- removed the D17 at (122.6, 308.2)
- removed the D17 at (183.4, 198.2)
- removed the D17 at (183.4, 308.2)
- removed the D2 at (79.9, 246.3)
- removed the D2 at (79.9, 136.3)
- removed the D2 at (226.2, 136.3)
- removed the D2 at (226.2, 246.3)
- removed the D3 at (97.8, 135.0)
- removed the D3 at (97.8, 245.0)
- removed the D3 at (208.3, 245.0)
- removed the D3 at (208.3, 135.0)
- removed the D4 at (116.7, 250.0)
- removed the D4 at (116.7, 140.0)
- removed the D4 at (189.4, 250.0)
- removed the D4 at (189.4, 140.0)
- removed the D5 at (119.9, 247.4)
- removed the D5 at (119.9, 137.4)
- removed the D5 at (186.1, 137.4)
- removed the D5 at (186.1, 247.4)
- removed the D6 at (61.4, 267.5)
- removed the D6 at (61.4, 157.5)
- removed the D6 at (244.7, 267.5)
- removed the D6 at (244.7, 157.5)
- removed the D7 at (79.9, 154.5)
- removed the D7 at (79.9, 264.5)
- removed the D7 at (226.2, 264.5)
- removed the D7 at (226.2, 154.5)
- removed the D8 at (97.8, 151.7)
- removed the D8 at (97.8, 261.7)
- removed the D8 at (208.3, 151.7)
- removed the D8 at (208.3, 261.7)
- removed the D9 at (116.4, 156.9)
- removed the D9 at (116.4, 266.9)
- removed the D9 at (189.7, 266.9)
- removed the D9 at (189.7, 156.9)
- removed the SW1 at (253.0, 138.4)
- removed the SW1 at (53.0, 138.4)
- removed the SW1 at (53.0, 248.4)
- removed the SW1 at (253.0, 248.4)
- removed the SW1 at (253.0, 38.4)
- removed the SW10 at (178.7, 267.7)
- removed the SW10 at (127.4, 267.7)
- removed the SW10 at (178.7, 157.7)
- removed the SW10 at (127.4, 157.7)
- removed the SW10 at (178.7, 57.7)
- removed the SW11 at (253.8, 283.5)
- removed the SW11 at (52.2, 173.5)
- removed the SW11 at (52.2, 283.5)
- removed the SW11 at (253.8, 173.5)
- removed the SW11 at (253.8, 73.5)
- removed the SW12 at (234.7, 279.7)
- removed the SW12 at (234.7, 169.7)
- removed the SW12 at (71.3, 169.7)
- removed the SW12 at (71.3, 279.7)
- removed the SW12 at (234.7, 69.7)
- removed the SW13 at (89.6, 166.9)
- removed the SW13 at (89.6, 276.9)
- removed the SW13 at (216.4, 166.9)
- removed the SW13 at (216.4, 276.9)
- removed the SW13 at (216.4, 66.9)
- removed the SW14 at (197.4, 168.7)
- removed the SW14 at (108.7, 278.7)
- removed the SW14 at (108.7, 168.7)
- removed the SW14 at (197.4, 278.7)
- removed the SW14 at (197.4, 68.7)
- removed the SW15 at (126.7, 284.7)
- removed the SW15 at (179.4, 284.7)
- removed the SW15 at (126.7, 174.7)
- removed the SW15 at (179.4, 174.7)
- removed the SW15 at (179.4, 74.7)
- removed the SW16 at (111.4, 194.5)
- removed the SW16 at (194.7, 304.5)
- removed the SW16 at (111.4, 304.5)
- removed the SW16 at (194.7, 194.5)
- removed the SW16 at (194.7, 94.5)
- removed the SW17 at (130.8, 198.4)
- removed the SW17 at (175.3, 308.4)
- removed the SW17 at (130.8, 308.4)
- removed the SW17 at (175.3, 198.4)
- removed the SW17 at (175.3, 98.4)
- removed the SW2 at (71.3, 244.5)
- removed the SW2 at (71.3, 134.5)
- removed the SW2 at (234.7, 244.5)
- removed the SW2 at (234.7, 134.5)
- removed the SW2 at (234.7, 34.5)
- removed the SW3 at (216.4, 132.9)
- removed the SW3 at (216.4, 242.9)
- removed the SW3 at (89.6, 242.9)
- removed the SW3 at (89.6, 132.9)
- removed the SW3 at (216.4, 32.9)
- removed the SW4 at (196.5, 244.7)
- removed the SW4 at (109.6, 134.7)
- removed the SW4 at (109.6, 244.7)
- removed the SW4 at (196.5, 134.7)
- removed the SW4 at (196.5, 34.7)
- removed the SW5 at (128.0, 250.7)
- removed the SW5 at (178.1, 140.7)
- removed the SW5 at (178.1, 250.7)
- removed the SW5 at (128.0, 140.7)
- removed the SW5 at (178.1, 40.7)
- removed the SW6 at (253.8, 156.2)
- removed the SW6 at (52.2, 156.2)
- removed the SW6 at (52.2, 266.2)
- removed the SW6 at (253.8, 266.2)
- removed the SW6 at (253.8, 56.2)
- removed the SW7 at (234.7, 262.7)
- removed the SW7 at (71.3, 262.7)
- removed the SW7 at (234.7, 152.7)
- removed the SW7 at (71.3, 152.7)
- removed the SW7 at (234.7, 52.7)
- removed the SW8 at (89.6, 259.9)
- removed the SW8 at (89.6, 149.9)
- removed the SW8 at (216.4, 259.9)
- removed the SW8 at (216.4, 149.9)
- removed the SW8 at (216.4, 49.9)
- removed the SW9 at (196.9, 261.7)
- removed the SW9 at (196.9, 151.7)
- removed the SW9 at (109.1, 261.7)
- removed the SW9 at (109.1, 151.7)
- removed the SW9 at (196.9, 51.7)
- removed the TH1 at (60.6, 237.9)
- removed the TH1 at (60.6, 127.9)
- removed the TH1 at (245.5, 27.9)
- removed the TH1 at (245.5, 127.9)
- removed the TH1 at (245.5, 237.9)
- removed the TH2 at (120.8, 129.8)
- removed the TH2 at (120.8, 239.8)
- removed the TH2 at (185.3, 129.8)
- removed the TH2 at (185.3, 29.8)
- removed the TH2 at (185.3, 239.8)
- removed the TH3 at (64.3, 291.0)
- removed the TH3 at (64.3, 181.0)
- removed the TH3 at (241.7, 81.0)
- removed the TH3 at (241.7, 181.0)
- removed the TH3 at (241.7, 291.0)
- removed the TH4 at (122.7, 188.6)
- removed the TH4 at (122.7, 298.6)
- removed the TH4 at (183.4, 88.6)
- removed the TH4 at (183.4, 188.6)
- removed the TH4 at (183.4, 298.6)
- removed the U1 at (58.9, 303.6)
- removed the U1 at (58.9, 193.6)
- removed the U1 at (247.2, 193.6)
- removed the U1 at (247.2, 303.6)
- added Batt_Hole_1: HOLE, jw_custom_footprints:MountingHole_2.2mm_M2_cutout, F.Cu at (223.4, 206.8)
- added Batt_Hole_1: HOLE, jw_custom_footprints:MountingHole_2.2mm_M2_cutout, F.Cu at (61.5, 205.0)
- added Batt_Hole_2: HOLE, jw_custom_footprints:MountingHole_2.2mm_M2_cutout, F.Cu at (201.1, 203.9)
- added Batt_Hole_2: HOLE, jw_custom_footprints:MountingHole_2.2mm_M2_cutout, F.Cu at (83.8, 202.0)
- added D1: D, jw_custom_footprints:Diode_SOD123_THT_2_cutout_small, F.Cu at (48.0, 144.5)
- added D1: D, jw_custom_footprints:Diode_SOD123_THT_2_cutout_small, B.Cu at (237.0, 146.3)
- added D10: D, jw_custom_footprints:Diode_SOD123_THT_2_cutout_small, F.Cu at (121.3, 170.2)
- added D10: D, jw_custom_footprints:Diode_SOD123_THT_2_cutout_small, B.Cu at (163.6, 172.0)
- added D11: D, jw_custom_footprints:Diode_SOD123_THT_2_cutout_small, F.Cu at (48.0, 182.4)
- added D11: D, jw_custom_footprints:Diode_SOD123_THT_2_cutout_small, B.Cu at (237.0, 184.2)
- added D12: D, jw_custom_footprints:Diode_SOD123_THT_2_cutout_small, F.Cu at (66.5, 179.1)
- added D12: D, jw_custom_footprints:Diode_SOD123_THT_2_cutout_small, B.Cu at (218.5, 180.9)
- added D13: D, jw_custom_footprints:Diode_SOD123_THT_2_cutout_small, F.Cu at (84.4, 176.4)
- added D13: D, jw_custom_footprints:Diode_SOD123_THT_2_cutout_small, B.Cu at (200.5, 178.2)
- added D14: D, jw_custom_footprints:Diode_SOD123_THT_2_cutout_small, F.Cu at (102.8, 181.4)
- added D14: D, jw_custom_footprints:Diode_SOD123_THT_2_cutout_small, B.Cu at (182.1, 183.3)
- added D15: D, jw_custom_footprints:Diode_SOD123_THT_2_cutout_small, F.Cu at (121.2, 186.7)
- added D15: D, jw_custom_footprints:Diode_SOD123_THT_2_cutout_small, B.Cu at (163.7, 188.5)
- added D16: D, jw_custom_footprints:Diode_SOD123_THT_2_cutout_small, F.Cu at (106.2, 205.4)
- added D16: D, jw_custom_footprints:Diode_SOD123_THT_2_cutout_small, B.Cu at (178.7, 207.2)
- added D17: D, jw_custom_footprints:Diode_SOD123_THT_2_cutout_small, F.Cu at (109.2, 205.9)
- added D17: D, jw_custom_footprints:Diode_SOD123_THT_2_cutout_small, B.Cu at (175.7, 207.7)
- added D2: D, jw_custom_footprints:Diode_SOD123_THT_2_cutout_small, F.Cu at (66.5, 144.5)
- added D2: D, jw_custom_footprints:Diode_SOD123_THT_2_cutout_small, B.Cu at (218.5, 146.4)
- added D3: D, jw_custom_footprints:Diode_SOD123_THT_2_cutout_small, F.Cu at (84.4, 142.7)
- added D3: D, jw_custom_footprints:Diode_SOD123_THT_2_cutout_small, B.Cu at (200.5, 144.5)
- added D4: D, jw_custom_footprints:Diode_SOD123_THT_2_cutout_small, F.Cu at (103.3, 147.7)
- added D4: D, jw_custom_footprints:Diode_SOD123_THT_2_cutout_small, B.Cu at (181.6, 149.5)
- added D5: D, jw_custom_footprints:Diode_SOD123_THT_2_cutout_small, F.Cu at (106.5, 145.1)
- added D5: D, jw_custom_footprints:Diode_SOD123_THT_2_cutout_small, B.Cu at (178.4, 146.9)
- added D6: D, jw_custom_footprints:Diode_SOD123_THT_2_cutout_small, F.Cu at (47.6, 165.1)
- added D6: D, jw_custom_footprints:Diode_SOD123_THT_2_cutout_small, B.Cu at (237.3, 167.0)
- added D7: D, jw_custom_footprints:Diode_SOD123_THT_2_cutout_small, F.Cu at (66.5, 162.2)
- added D7: D, jw_custom_footprints:Diode_SOD123_THT_2_cutout_small, B.Cu at (218.5, 164.0)
- added D8: D, jw_custom_footprints:Diode_SOD123_THT_2_cutout_small, F.Cu at (84.4, 159.4)
- added D8: D, jw_custom_footprints:Diode_SOD123_THT_2_cutout_small, B.Cu at (200.5, 161.3)
- added D9: D, jw_custom_footprints:Diode_SOD123_THT_2_cutout_small, F.Cu at (103.0, 164.7)
- added D9: D, jw_custom_footprints:Diode_SOD123_THT_2_cutout_small, B.Cu at (181.9, 166.5)
- added PWR_SW_3: SW_DPDT, jw_custom_footprints:Button_Switch_Push_Vertical_2P2T_Toggle_5.8x5.8_cutout, F.Cu at (125.3, 94.4)
- added PWR_SW_3: SW_DPDT, jw_custom_footprints:Button_Switch_Push_Vertical_2P2T_Toggle_5.8x5.8_cutout, B.Cu at (159.6, 96.2)
- added SW1: SW1, jw_custom_footprints:Kailh_socket_PG1350_v1_reversible_cutout_bottom_alt, F.Cu at (245.3, 147.9)
- added SW1: SW1, jw_custom_footprints:Kailh_socket_PG1350_v1_reversible_cutout_bottom_alt, F.Cu at (39.6, 146.1)
- added SW1: SW1, jw_custom_footprints:Kailh_socket_PG1350_v1_reversible_cutout_14x14mm, B.Cu at (245.3, 47.9)
- added SW10: SW10, jw_custom_footprints:Kailh_socket_PG1350_v1_reversible_cutout_bottom_alt, F.Cu at (114.0, 165.4)
- added SW10: SW10, jw_custom_footprints:Kailh_socket_PG1350_v1_reversible_cutout_bottom_alt, F.Cu at (170.9, 167.2)
- added SW10: SW10, jw_custom_footprints:Kailh_socket_PG1350_v1_reversible_cutout_14x14mm, B.Cu at (170.9, 67.2)
- added SW11: SW11, jw_custom_footprints:Kailh_socket_PG1350_v1_reversible_cutout_bottom_alt, F.Cu at (38.8, 181.2)
- added SW11: SW11, jw_custom_footprints:Kailh_socket_PG1350_v1_reversible_cutout_bottom_alt, F.Cu at (246.1, 183.0)
- added SW11: SW11, jw_custom_footprints:Kailh_socket_PG1350_v1_reversible_cutout_14x14mm, B.Cu at (246.1, 83.0)
- added SW12: SW12, jw_custom_footprints:Kailh_socket_PG1350_v1_reversible_cutout_bottom_alt, F.Cu at (227.0, 179.2)
- added SW12: SW12, jw_custom_footprints:Kailh_socket_PG1350_v1_reversible_cutout_bottom_alt, F.Cu at (57.9, 177.4)
- added SW12: SW12, jw_custom_footprints:Kailh_socket_PG1350_v1_reversible_cutout_14x14mm, B.Cu at (227.0, 79.2)
- added SW13: SW13, jw_custom_footprints:Kailh_socket_PG1350_v1_reversible_cutout_bottom_alt, F.Cu at (208.7, 176.4)
- added SW13: SW13, jw_custom_footprints:Kailh_socket_PG1350_v1_reversible_cutout_bottom_alt, F.Cu at (76.2, 174.6)
- added SW13: SW13, jw_custom_footprints:Kailh_socket_PG1350_v1_reversible_cutout_14x14mm, B.Cu at (208.7, 76.4)
- added SW14: SW14, jw_custom_footprints:Kailh_socket_PG1350_v1_reversible_cutout_bottom_alt, F.Cu at (95.3, 176.4)
- added SW14: SW14, jw_custom_footprints:Kailh_socket_PG1350_v1_reversible_cutout_bottom_alt, F.Cu at (189.6, 178.2)
- added SW14: SW14, jw_custom_footprints:Kailh_socket_PG1350_v1_reversible_cutout_14x14mm, B.Cu at (189.6, 78.2)
- added SW15: SW15, jw_custom_footprints:Kailh_socket_PG1350_v1_reversible_cutout_bottom_alt, F.Cu at (113.2, 182.4)
- added SW15: SW15, jw_custom_footprints:Kailh_socket_PG1350_v1_reversible_cutout_bottom_alt, F.Cu at (171.7, 184.2)
- added SW15: SW15, jw_custom_footprints:Kailh_socket_PG1350_v1_reversible_cutout_14x14mm, B.Cu at (171.7, 84.2)
- added SW16: SW16, jw_custom_footprints:Kailh_socket_PG1350_v1_reversible_cutout_bottom_alt, F.Cu at (98.0, 202.2)
- added SW16: SW16, jw_custom_footprints:Kailh_socket_PG1350_v1_reversible_cutout_bottom_alt, F.Cu at (186.9, 204.0)
- added SW16: SW16, jw_custom_footprints:Kailh_socket_PG1350_v1_reversible_cutout_14x14mm, B.Cu at (186.9, 104.0)
- added SW17: SW17, jw_custom_footprints:Kailh_socket_PG1350_v1_reversible_cutout_bottom_alt, F.Cu at (167.5, 207.9)
- added SW17: SW17, jw_custom_footprints:Kailh_socket_PG1350_v1_reversible_cutout_bottom_alt, F.Cu at (117.4, 206.1)
- added SW17: SW17, jw_custom_footprints:Kailh_socket_PG1350_v1_reversible_cutout_14x14mm, B.Cu at (167.5, 107.9)
- added SW2: SW2, jw_custom_footprints:Kailh_socket_PG1350_v1_reversible_cutout_bottom_alt, F.Cu at (57.9, 142.7)
- added SW2: SW2, jw_custom_footprints:Kailh_socket_PG1350_v1_reversible_cutout_bottom_alt, F.Cu at (227.0, 144.5)
- added SW2: SW2, jw_custom_footprints:Kailh_socket_PG1350_v1_reversible_cutout_14x14mm, B.Cu at (227.0, 44.5)
- added SW3: SW3, jw_custom_footprints:Kailh_socket_PG1350_v1_reversible_cutout_bottom_alt, F.Cu at (208.7, 142.4)
- added SW3: SW3, jw_custom_footprints:Kailh_socket_PG1350_v1_reversible_cutout_bottom_alt, F.Cu at (76.2, 140.6)
- added SW3: SW3, jw_custom_footprints:Kailh_socket_PG1350_v1_reversible_cutout_14x14mm, B.Cu at (208.7, 42.4)
- added SW4: SW4, jw_custom_footprints:Kailh_socket_PG1350_v1_reversible_cutout_bottom_alt, F.Cu at (188.7, 144.2)
- added SW4: SW4, jw_custom_footprints:Kailh_socket_PG1350_v1_reversible_cutout_bottom_alt, F.Cu at (96.2, 142.4)
- added SW4: SW4, jw_custom_footprints:Kailh_socket_PG1350_v1_reversible_cutout_14x14mm, B.Cu at (188.7, 44.2)
- added SW5: SW5, jw_custom_footprints:Kailh_socket_PG1350_v1_reversible_cutout_bottom_alt, F.Cu at (114.6, 148.4)
- added SW5: SW5, jw_custom_footprints:Kailh_socket_PG1350_v1_reversible_cutout_bottom_alt, F.Cu at (170.3, 150.2)
- added SW5: SW5, jw_custom_footprints:Kailh_socket_PG1350_v1_reversible_cutout_14x14mm, B.Cu at (170.3, 50.2)
- added SW6: SW6, jw_custom_footprints:Kailh_socket_PG1350_v1_reversible_cutout_bottom_alt, F.Cu at (38.5, 163.8)
- added SW6: SW6, jw_custom_footprints:Kailh_socket_PG1350_v1_reversible_cutout_bottom_alt, F.Cu at (246.4, 165.6)
- added SW6: SW6, jw_custom_footprints:Kailh_socket_PG1350_v1_reversible_cutout_14x14mm, B.Cu at (246.4, 65.6)
- added SW7: SW7, jw_custom_footprints:Kailh_socket_PG1350_v1_reversible_cutout_bottom_alt, F.Cu at (227.0, 162.2)
- added SW7: SW7, jw_custom_footprints:Kailh_socket_PG1350_v1_reversible_cutout_bottom_alt, F.Cu at (57.9, 160.4)
- added SW7: SW7, jw_custom_footprints:Kailh_socket_PG1350_v1_reversible_cutout_14x14mm, B.Cu at (227.0, 62.2)
- added SW8: SW8, jw_custom_footprints:Kailh_socket_PG1350_v1_reversible_cutout_bottom_alt, F.Cu at (76.2, 157.6)
- added SW8: SW8, jw_custom_footprints:Kailh_socket_PG1350_v1_reversible_cutout_bottom_alt, F.Cu at (208.7, 159.4)
- added SW8: SW8, jw_custom_footprints:Kailh_socket_PG1350_v1_reversible_cutout_14x14mm, B.Cu at (208.7, 59.4)
- added SW9: SW9, jw_custom_footprints:Kailh_socket_PG1350_v1_reversible_cutout_bottom_alt, F.Cu at (95.7, 159.4)
- added SW9: SW9, jw_custom_footprints:Kailh_socket_PG1350_v1_reversible_cutout_bottom_alt, F.Cu at (189.2, 161.2)
- added SW9: SW9, jw_custom_footprints:Kailh_socket_PG1350_v1_reversible_cutout_14x14mm, B.Cu at (189.2, 61.2)
- added TH1: HOLE, jw_custom_footprints:MountingHole_2.2mm_M2_cutout, F.Cu at (47.2, 135.6)
- added TH1: HOLE, jw_custom_footprints:MountingHole_2.2mm_M2_cutout, B.Cu at (237.8, 37.4)
- added TH1: HOLE, jw_custom_footprints:MountingHole_2.2mm_M2_cutout, B.Cu at (237.8, 137.4)
- added TH2: HOLE, jw_custom_footprints:MountingHole_2.2mm_M2_cutout, F.Cu at (107.4, 137.5)
- added TH2: HOLE, jw_custom_footprints:MountingHole_2.2mm_M2_cutout, B.Cu at (177.5, 39.3)
- added TH2: HOLE, jw_custom_footprints:MountingHole_2.2mm_M2_cutout, B.Cu at (177.5, 139.3)
- added TH3: HOLE, jw_custom_footprints:MountingHole_2.2mm_M2_cutout, F.Cu at (50.9, 188.4)
- added TH3: HOLE, jw_custom_footprints:MountingHole_2.2mm_M2_cutout, B.Cu at (234.0, 90.2)
- added TH3: HOLE, jw_custom_footprints:MountingHole_2.2mm_M2_cutout, B.Cu at (234.0, 190.2)
- added TH4: HOLE, jw_custom_footprints:MountingHole_2.2mm_M2_cutout, F.Cu at (109.2, 196.3)
- added TH4: HOLE, jw_custom_footprints:MountingHole_2.2mm_M2_cutout, B.Cu at (175.7, 98.1)
- added TH4: HOLE, jw_custom_footprints:MountingHole_2.2mm_M2_cutout, B.Cu at (175.7, 198.1)
- added U1: SeeeduinoXIAO_nRF52840, jw_custom_footprints:Xiao_nRF52840_THT_jumper_1.55mm_hole_cutout_alt, F.Cu at (45.5, 201.3)
- added U1: SeeeduinoXIAO_nRF52840, jw_custom_footprints:Xiao_nRF52840_THT_jumper_1.55mm_hole_cutout_alt, B.Cu at (239.5, 203.1)
- moved SW2 15.7 mm to (57.9, 42.7)
- moved SW6 15.7 mm to (38.5, 63.8)
- moved SW15 15.5 mm to (113.2, 82.4)
- moved SW3 15.5 mm to (76.2, 40.6)
- moved SW8 15.5 mm to (76.2, 57.6)
- moved SW9 15.5 mm to (95.7, 59.4)
- moved TH2 15.5 mm to (107.4, 37.5)
- moved SW10 15.5 mm to (114.0, 65.4)
- moved SW13 15.5 mm to (76.2, 74.6)
- moved SW1 15.5 mm to (39.6, 46.1)
- moved TH1 15.5 mm to (47.2, 35.6)
- moved SW17 15.5 mm to (117.4, 106.1)
- moved TH4 15.5 mm to (109.2, 96.3)
- moved SW4 15.5 mm to (96.2, 42.4)
- moved SW7 15.5 mm to (57.9, 60.4)
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Other:
- board size 224.6 x 368.5 mm -> 230.2 x 191.4 mm
